File: Prj 4 - 4x8x4 Matrix Clock/Prj 4 - 4x8x4 Matrix Clock.kicad_sch (KiCad schematic)
At the start: 19 parts, among them J1 Barrel_Jack, J2 Conn_01x05_Pin, J3 Conn_01x05_Pin, J4 Conn_01x05_Pin, J5 Conn_01x05_Pin, J6 Conn_01x05_Pin, J7 Conn_01x05_Pin, J8 Conn_01x05_Pin, J9 Conn_01x05_Pin, U1 ARDUINO_PRO_MINI

Commit message: Update Prj 4 - 4x8x4 Matrix Clock.kicad_sch
Update text for git test
Other:
- note added: "These connectors are flipped vertically so that pin numbers correspond correctly acrooss all headers. BLIP!"
- note removed: "These connectors are flipped vertically so that pin numbers correspond correctly acrooss all headers"
Changed lines of the file:
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@@
 		)
 	)
-	(text "These connectors are flipped vertically\nso that pin numbers correspond correctly\nacrooss all headers"
+	(text "These connectors are flipped vertically\nso that pin numbers correspond correctly\nacrooss all headers. BLIP!"
 		(exclude_from_sim no)
 		(at 161.29 154.94 0)

Commit message: Update Prj 4 - 4x8x4 Matrix Clock.kicad_sch
Removed BLIP!
Other:
- note added: "These connectors are flipped vertically so that pin numbers correspond correctly acrooss all headers."
- note removed: "These connectors are flipped vertically so that pin numbers correspond correctly acrooss all headers. BLIP!"
Changed lines of the file:
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@@
 		)
 	)
-	(text "These connectors are flipped vertically\nso that pin numbers correspond correctly\nacrooss all headers. BLIP!"
+	(text "These connectors are flipped vertically\nso that pin numbers correspond correctly\nacrooss all headers."
 		(exclude_from_sim no)
 		(at 161.29 154.94 0)

Commit message: Update Prj 4 - 4x8x4 Matrix Clock.kicad_sch
Fixed typo
Other:
- note added: "These connectors are flipped vertically so that pin numbers correspond correctly accrooss all headers. <<-- Fixed typo!"
- note removed: "These connectors are flipped vertically so that pin numbers correspond correctly acrooss all headers."
Changed lines of the file:
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@@
 		)
 	)
-	(text "These connectors are flipped vertically\nso that pin numbers correspond correctly\nacrooss all headers."
+	(text "These connectors are flipped vertically\nso that pin numbers correspond correctly\naccrooss all headers. <<-- Fixed typo!"
 		(exclude_from_sim no)
 		(at 161.29 154.94 0)
